Commit message: fixed spurious homotopy class in wall

File: urdf/wall.urdf (robot description, URDF)
Before this commit: robot wall_description, 151 links, 150 joints
Links:
- added link box146; collision box size=0.270000 0.405009 0.250500; visual box size=0.170000 0.405009 0.050500
Joints:
- added joint base_to_box146: type fixed, parent base_link, child box146

Commit message: added free space computation interface

File: urdf/wall.urdf (robot description, URDF)
Before this commit: robot wall_description, 152 links, 151 joints
Links:
- removed link wall_back1
- removed link wall_back2
- removed link wall_left1
- removed link wall_left2
- removed link wall_right1
- removed link wall_right2
- link box146: geometry collision box size=0.250000 0.405009 0.250500; visual box size=0.300000 0.405009 0.250500
Joints:
- removed joint base_to_wall_back1
- removed joint base_to_wall_back2
- removed joint base_to_wall_left1
- removed joint base_to_wall_left2
- removed joint base_to_wall_right1
- removed joint base_to_wall_right2
